File: uEVSE/uEVSE.kicad_sch (KiCad schematic)
At the start: 33 parts, among them J1 PE PP CP, J2 PE PP CP, J3 Prog, J4 12VDCin, J5 12VDCin, U1 NE555P, U2 LM358, U3 TC4428xOA, U4 ESP-07, U6 R-783.3-1.0

Commit message: Add files via upload
Parts:
- removed C4: 100uF, symbol Device:C_Polarized
- removed J1: PE PP CP, symbol Connector:Screw_Terminal_01x03
- removed J5: 12VDCin, symbol Connector:Screw_Terminal_01x02
- removed JP2: SolderJumper_2_Bridged, symbol Jumper:SolderJumper_2_Bridged
- removed R2: 1k, symbol Device:R
- removed R3: R, symbol Device:R
- added J1, J5, J6, J7, J8: GSsP, Connector_PinHeader_2.54mm:PinHeader_1x04_P2.54mm_Vertical, symbol Connector:Conn_01x04_Pin
- added J10: Conn_02x04_Odd_Even, symbol Connector_Generic:Conn_02x04_Odd_Even
- added J9: Conn_02x04_Counter_Clockwise, symbol Connector_Generic:Conn_02x04_Counter_Clockwise
- added JP2: SolderJumper_2_Open, Jumper:SolderJumper-2_P1.3mm_Open_RoundedPad1.0x1.5mm, symbol Jumper:SolderJumper_2_Open
- C10, C2, C3, C6: footprint (none) -> Capacitor_THT:C_Axial_L5.1mm_D3.1mm_P7.50mm_Horizontal
- C5, C8: footprint (none) -> Capacitor_THT:CP_Radial_D7.5mm_P2.50mm
- C7: value 47uF -> 100uF; footprint (none) -> Capacitor_THT:CP_Radial_D7.5mm_P2.50mm
- D1, D2: value D -> 1N4148; footprint (none) -> Diode_THT:D_A-405_P2.54mm_Vertical_AnodeUp
- J2: footprint (none) -> TerminalBlock:TerminalBlock_bornier-3_P5.08mm
- J3: footprint (none) -> Connector_PinHeader_2.54mm:PinHeader_1x04_P2.54mm_Vertical
- J4: footprint (none) -> TerminalBlock:TerminalBlock_bornier-2_P5.08mm
- JP1: footprint (none) -> Jumper:SolderJumper-2_P1.3mm_Bridged_RoundedPad1.0x1.5mm
- R1, R6, R8, R9: footprint (none) -> Resistor_THT:R_Axial_DIN0207_L6.3mm_D2.5mm_P2.54mm_Vertical
- R4: value R -> 10k; footprint (none) -> Resistor_THT:R_Axial_DIN0207_L6.3mm_D2.5mm_P2.54mm_Vertical
- R5: value R -> 100k; footprint (none) -> Resistor_THT:R_Axial_DIN0207_L6.3mm_D2.5mm_P2.54mm_Vertical
- RV1: renamed from RV2; value Delay -> 100k; footprint (none) -> Potentiometer_THT:Potentiometer_Bourns_3266Y_Vertical
- RV2: renamed from RV4; value Freq -> 10k; footprint (none) -> Potentiometer_THT:Potentiometer_Bourns_3266Y_Vertical
- RV3: value Duty -> 100k; footprint (none) -> Potentiometer_THT:Potentiometer_Bourns_3266Y_Vertical
- U2: footprint (none) -> Package_DIP:DIP-8_W7.62mm
- U3: footprint Package_SO:SOIC-8_3.9x4.9mm_P1.27mm -> Package_DIP:DIP-8_W7.62mm
Connections:
- net +12V: now also RV1.3, J1.4 (Pin_4), J5.4 (Pin_4), J6.4 (Pin_4), J7.4 (Pin_4), J8.4 (Pin_4); no longer RV1.1
- net GNDD: now also RV1.1, J1.1 (Pin_1), J5.1 (Pin_1), J6.1 (Pin_1), J7.1 (Pin_1), J8.1 (Pin_1); no longer C3.1, C7.1, RV1.3, U4.1 (~{RST}), U4.3 (EN), U4.8 (VCC), U6.3 (OUT)
- net at U3.7 (~{OUT_A}): now also J7.3 (Pin_3)
- net at U3.5 (OUT_B): now also J7.2 (Pin_2)
- net at J3.4 (Pin_4), U4.12 (GPIO0): now also J1.3 (Pin_3)
- net at U1.3 (Q), U2.2 (-): now also J5.3 (Pin_3); no longer R8.1
- net at J2.1 (Pin_1), JP1.2 (B), R9.2: now also J8.3 (Pin_3); no longer U2.1
- new net: J5.2 (Pin_2), U2.1
- new net: J6.2 (Pin_2), JP2.1 (A), U3.4 (IN_B)
- new net: J6.3 (Pin_3), JP2.2 (B), U3.2 (IN_A)
- new net: J8.2 (Pin_2), R8.1
- new net: C3.1, C7.1, U4.1 (~{RST}), U4.3 (EN), U4.8 (VCC), U6.3 (OUT)
- new net: J1.2 (Pin_2), U4.11 (GPIO2)
Other:
- moved on the sheet: C8, J2, J3, J4, JP1, R8, R9, U2C, U3
