File: uEVSE.kicad_pcb (KiCad board)
At the start: 2 copper layers, 81.9 x 10.5 mm, 25 parts, among them J1 12VDC input, J2 GSsP, J3 PE/CP, J4 Ss(B), U1 NE555P, U2 LM358

Commit message: Add files via upload
Parts:
- added C4: 4.7nF, Capacitor_THT:C_Rect_L7.0mm_W2.5mm_P5.00mm, F.Cu at (79.9, 98.3)
- moved C2 2.37 mm to (79.9, 101.4)
- moved C6 0.76 mm to (80.0, 104.9)
Routing:
- net Net-(U1-R): track 53.6 -> 58.3 mm
- net +12V: track 102.6 -> 106.1 mm
- net Net-(U1-THR): track 37.2 -> 39.4 mm
- net GNDD: track 105.0 -> 107.0 mm
- net Net-(J2-Pin_3): track 40.1 -> 41.0 mm
Other:
- board text added: "+12V-"
- board text added: "CP"
- board text added: "PE"
- board text added: "PE CP"
